Commit message: right wheel

File: urdf/box_bot_geometric.urdf (robot description, URDF)
Before this commit: robot box_bot, 3 links, 2 joints
Links:
- added link right_wheel; visual cylinder length=0.001 radius=0.035
Joints:
- added joint right_wheel: type continuous, parent chassis, child right_wheel, origin xyz=0.0 -0.05 -0.025 rpy=0 0 0, axis 0 1 0, limit effort=10000 velocity=1000

Commit message: casters

File: urdf/box_bot_geometric.urdf (robot description, URDF)
Before this commit: robot box_bot, 4 links, 3 joints
Links:
- added link back_pitch_link; visual sphere radius=0.010
- added link back_roll_link; visual cylinder length=0.005 radius=0.010
- added link back_yaw_link; visual cylinder length=0.005 radius=0.010
- added link front_pitch_link; visual sphere radius=0.010
- added link front_roll_link; visual cylinder length=0.005 radius=0.010
- added link front_yaw_link; visual cylinder length=0.005 radius=0.010
Joints:
- added joint back_pitch_joint: type continuous, parent back_roll_link, child back_pitch_link, origin xyz=0 0 0 rpy=0 0 0, axis 0 1 0, limit effort=10000 velocity=1000
- added joint back_roll_joint: type continuous, parent back_yaw_link, child back_roll_link, origin xyz=0 0 0 rpy=0 0 0, axis 1 0 0, limit effort=10000 velocity=1000
- added joint back_yaw_joint: type continuous, parent chassis, child back_yaw_link, origin xyz=-0.04 0 -0.05 rpy=0 0 0, axis 0 0 1, limit effort=10000 velocity=1000
- added joint front_pitch_joint: type continuous, parent front_roll_link, child front_pitch_link, origin xyz=0 0 0 rpy=0 0 0, axis 0 1 0, limit effort=10000 velocity=1000
- added joint front_roll_joint: type continuous, parent front_yaw_link, child front_roll_link, origin xyz=0 0 0 rpy=0 0 0, axis 1 0 0, limit effort=10000 velocity=1000
- added joint front_yaw_joint: type continuous, parent chassis, child front_yaw_link, origin xyz=0.04 0 -0.05 rpy=0 0 0, axis 0 0 1, limit effort=10000 velocity=1000
