Commit message: resizing caster cylinders
Cylinders were used to get additional degrees of freedom for the caster,
but they should be small so as not to collide with the environment.

File: urdf/box_bot_geometric_meshes_collisions_inertias.urdf (robot description, URDF)
Before this commit: robot box_bot, 10 links, 9 joints
Links:
- link back_roll_link: geometry visual cylinder length=0.001 radius=0.0045000000000000005
- link back_yaw_link: geometry visual cylinder length=0.001 radius=0.0045000000000000005
- link front_roll_link: geometry visual cylinder length=0.001 radius=0.0045000000000000005
- link front_yaw_link: geometry visual cylinder length=0.001 radius=0.0045000000000000005
