Commit message: fixed error from wheels and wheel joints have duplicate names

File: urdf/box_bot_meshes_collisions_inertias.urdf (robot description, URDF)
Before this commit: robot box_bot, 10 links, 9 joints
Joints:
- removed joint left_wheel
- removed joint right_wheel
- added joint left_wheel_joint: type continuous, parent chassis, child left_wheel, origin xyz=0.0 0.05 -0.025 rpy=0 0 0, axis 0 1 0, limit effort=10000 velocity=1000
- added joint right_wheel_joint: type continuous, parent chassis, child right_wheel, origin xyz=0.0 -0.05 -0.025 rpy=0 0 0, axis 0 1 0, limit effort=10000 velocity=1000
