Commit message: spawning and operating two robots from the same model

File: urdf/box_bot.xacro (robot description, xacro)
@@ -1,4 +1,5 @@
 <?xml version="1.0"?>
 <robot xmlns:xacro="http://www.ros.org/wiki/xacro" name="box_bot">
+<xacro:property name="robot_name" value="$(arg robot_name)"/>
 <xacro:include filename="$(find box_bot_description)/urdf/box_bot.gazebo.xacro" />
 <xacro:gazebo_elements />
@@ -27,5 +28,5 @@
     </inertial>
   </link>
-  <!-- XACRO: Wheel macro -->'
+  <!-- XACRO: Wheel macro -->
   <xacro:macro name="wheel" params="wheel_name">
     <link name="${wheel_name}">
@@ -240,3 +241,46 @@
     <dynamics damping="0.0" friction="0.1"/>
   </joint>
+    <!-- PLUGINS -->
+  <!-- JOINT PUBLISHER -->
+  <gazebo>
+    <plugin name="box_bot_joint_state" filename="libgazebo_ros_joint_state_publisher.so">
+      <ros>
+        <namespace>/${robot_name}</namespace>
+          <remapping>~/out:=joint_states</remapping>
+      </ros>
+      <update_rate>30</update_rate>
+      <joint_name>joint_left_wheel</joint_name>
+      <joint_name>joint_right_wheel</joint_name>
+      <joint_name>front_yaw_joint</joint_name>
+      <joint_name>back_yaw_joint</joint_name>
+      <joint_name>front_roll_joint</joint_name>
+      <joint_name>back_roll_joint</joint_name>
+      <joint_name>front_pitch_joint</joint_name>
+      <joint_name>back_pitch_joint</joint_name>
+    </plugin>
+  </gazebo>
+  <!-- Differential drive -->
+  <gazebo>
+    <plugin filename="libgazebo_ros_diff_drive.so" name="differential_drive_controller">
+      <ros>
+        <namespace>/${robot_name}</namespace>
+          <remapping>/cmd_vel:=cmd_vel</remapping>
+      </ros>
+      <!-- wheels -->
+      <left_joint>joint_left_wheel</left_joint>
+      <right_joint>joint_right_wheel</right_joint>
+      <!-- kinematics -->
+      <wheel_separation>0.1</wheel_separation>
+      <wheel_diameter>0.07</wheel_diameter>
+      <!-- limits -->
+      <max_wheel_torque>1.0</max_wheel_torque>
+      <max_wheel_acceleration>2.0</max_wheel_acceleration>
+      <!-- output -->
+      <publish_odom>true</publish_odom>
+      <publish_odom_tf>true</publish_odom_tf>
+      <!-- TF frames -->
+      <odometry_frame>${robot_name}/odom</odometry_frame>
+      <robot_base_frame>${robot_name}/base_link</robot_base_frame>
+    </plugin>
+  </gazebo>
 </robot>
