Commit message: added point-cloud sensor plugin

File: urdf/box_bot_final.urdf (robot description, URDF)
Before this commit: robot box_bot, 13 links, 12 joints
Links:
- added link pointcloud_link
Joints:
- added joint pointcloud_link_joint: type fixed, parent chassis, child pointcloud_link, origin xyz=0.051 0.0 0 rpy=0 0 0, axis 0 0 0

Commit message: added rgb camera

File: urdf/box_bot_final.urdf (robot description, URDF)
Before this commit: robot box_bot, 14 links, 13 joints
Links:
- added link rgb_camera_link_frame
Joints:
- added joint rgb_camera_link_frame_joint: type fixed, parent chassis, child rgb_camera_link_frame, origin xyz=0.051 0.0 0.05 rpy=0 0 0, axis 0 0 0

Commit message: adding regular camera

File: urdf/box_bot_final.urdf (robot description, URDF)
Before this commit: robot box_bot, 15 links, 14 joints
Links:
- added link camera_link
Joints:
- added joint camera_joint: type fixed, parent base_link, child camera_link, origin xyz=0.0 0.0 0.2 rpy=0 0 0

Commit message: adding IMU

File: urdf/box_bot_final.urdf (robot description, URDF)
Before this commit: robot box_bot, 16 links, 15 joints
Links:
- added link imu_link
Joints:
- added joint imu_joint: type fixed, parent base_link, child imu_link, origin xyz=-0.10 0 0.05 rpy=0 0 0

Commit message: moved sensors from base_link to chassis

File: urdf/box_bot_final.urdf (robot description, URDF)
Before this commit: robot box_bot, 17 links, 16 joints
Joints:
- joint camera_joint: parent base_link -> chassis
- joint imu_joint: parent base_link -> chassis
