Commit message: fixed poses of IMU and regular camera

File: urdf/box_bot_final_course_version.urdf (robot description, URDF)
Before this commit: robot box_bot, 17 links, 16 joints
Links:
- removed link camera_link
- removed link imu_link
- link chassis: geometry collision box size=0.1 0.1 0.1; visual mesh filename=package://my_box_bot_description/meshes/cute_cube.dae scale=0.1 0.1 0.1
- link laser_scan_model_link: geometry collision cylinder length=0.0408 radius=0.037493; visual mesh filename=package://my_box_bot_description/meshes/sensors/rplidar.dae scale=1.0 1.0 1.0
Joints:
- removed joint camera_joint
- removed joint imu_joint
